File: MP2759.kicad_sch (KiCad schematic)
At the start: 24 parts, among them U3 MP2759

Commit message: More fixes
Parts:
- D5, TH2: FT Rotation Offset (none) -> 180
- U3: FT Rotation Offset (none) -> -90
Changed lines of the file:
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@@
+			)
+		)
+		(property "FT Rotation Offset" "180"
+			(at 193.04 110.49 0)
+			(effects
+				(font
+					(size 1.27 1.27)
+				)
+				(hide yes)
 			)
 		)
@@
 			)
 		)
+		(property "FT Rotation Offset" "-90"
+			(at 168.91 85.09 0)
+			(effects
+				(font
+					(size 1.27 1.27)
+				)
+				(hide yes)
+			)
+		)
 		(pin "4"
 		)
@@
 			(at 49.53 93.98 90)
 			(effects
+				(font
+					(size 1.27 1.27)
+				)
+				(hide yes)
+			)
+		)
+		(property "FT Rotation Offset" "180"
+			(at 49.53 93.98 90)
+			(effects

Commit message: Set LED resistors
Parts:
- R21: value R -> 16k
- R22: value R -> 4.7k
Changed lines of the file:
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@@
 			)
 		)
-		(property "Value" "R"
+		(property "Value" "4.7k"
 			(at 90.17 166.3699 0)
 			(effects
@@
 		(fields_autoplaced yes)
 		(property "Reference" "R21"
-			(at 74.93 163.83 0)
+			(at 74.93 163.8299 0)
 			(effects
 				(font
@@
 			)
 		)
-		(property "Value" "R"
-			(at 74.93 166.37 0)
-			(effects
-				(font
+		(property "Value" "16k"
+			(at 74.93 166.3699 0)
+			(effects
+				(font

Commit message: Switch to JST-PH connectors Add Sheet titles
Parts:
- TH2: footprint Connector_JST:JST_ZH_B2B-ZR_1x02_P1.50mm_Vertical -> Connector_JST:JST_PH_B2B-PH-K_1x02_P2.00mm_Vertical
Other:
- note added: "Use 103AT-2 thermistor JST-PH 2.0mm 2-pin connector"
- note removed: "Use 103AT-2 thermistor"
- title: (none) -> MP2759 Buck Charger
Changed lines of the file:
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@@
 	(paper "A4")
 	(title_block
+		(title "MP2759 Buck Charger")
 		(rev "1.0")
+		(comment 1 "Through-hole connectors not to be installed as part of PCBA")
+		(comment 2 "15-32V Input 3A max, reduced charge current below 18V")
 	)
 	(text "~3A Charge limit\n3A Input limit"
@@
 		)
 	)
-	(text "Use 103AT-2 thermistor"
+	(text "Use 103AT-2 thermistor\nJST-PH 2.0mm 2-pin connector"
 		(exclude_from_sim no)
-		(at 208.026 116.078 0)
+		(at 195.834 115.57 0)
 		(effects
 			(font
 				(size 1.27 1.27)
 			)
+			(justify left)
 		)
 	)
@@
 			)
 		)
-		(property "Footprint" "Connector_JST:JST_ZH_B2B-ZR_1x02_P1.50mm_Vertical"
+		(property "Footprint" "Connector_JST:JST_PH_B2B-PH-K_1x02_P2.00mm_Vertical"
 			(at 193.04 109.22 0)
 			(effects

Commit message: Action review feedback
Other:
- note added: "12V UVLO Current limiting <18V Note: Battery will not fully charge below 15V"
- note removed: "12V UVLO Current limiting <18V"
Changed lines of the file:
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@@
 		)
 	)
-	(text "12V UVLO\nCurrent limiting <18V"
+	(text "12V UVLO\nCurrent limiting <18V\n\nNote: Battery will not \nfully charge below 15V"
 		(exclude_from_sim no)
-		(at 96.012 108.966 0)
+		(at 96.52 110.49 0)
 		(effects
 			(font
