File: I2C_ctrl.kicad_sch (KiCad schematic)
At the start: 32 parts, among them J6 TYPE-C16PIN, J7 TagConnect 2030-NL, SW1 MS-22C01-G010, SW2 TS-1088-AR02016, U4 ATtiny1616-M, U5 CH340X, U6 ADuM1201AR, U7 SN74LVC1G3157, U8 SN74LVC1G3157

Commit message: More fixes
Parts:
- D3, D4: footprint Diode_SMD:D_SOD-123 -> Diode_SMD:D_SOD-323
- D6: FT Rotation Offset (none) -> 90
- U4: FT Rotation Offset (none) -> -90
- U7, U8: FT Rotation Offset (none) -> 180
Changed lines of the file:
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@@
 			)
 		)
+		(property "FT Rotation Offset" "180"
+			(at 217.17 140.97 0)
+			(effects
+				(font
+					(size 1.27 1.27)
+				)
+				(hide yes)
+			)
+		)
 		(pin "6"
 		)
@@
 			)
 		)
+		(property "FT Rotation Offset" "180"
+			(at 160.02 69.85 0)
+			(effects
+				(font
+					(size 1.27 1.27)
+				)
+				(hide yes)
+			)
+		)
 		(pin "6"
 		)
@@
 			)
 		)
+		(property "FT Rotation Offset" "180"
+			(at 160.02 52.07 0)
+			(effects
+				(font
+					(size 1.27 1.27)
+				)
+				(hide yes)
+			)
+		)
 		(pin "6"
 		)
@@
 			)
 		)
+		(property "FT Rotation Offset" "90"
+			(at 54.61 88.9 0)
+			(effects
+				(font
+					(size 1.27 1.27)
+				)
+				(hide yes)
+			)
+		)
 		(pin "4"
 		)
@@
 			)
 		)
-		(property "Footprint" "Diode_SMD:D_SOD-123"
+		(property "Footprint" "Diode_SMD:D_SOD-323"
 			(at 162.56 116.84 90)
 			(effects
@@
 			)
 		)
+		(property "FT Rotation Offset" "180"
+			(at 227.33 140.97 0)
+			(effects
+				(font
+					(size 1.27 1.27)
+				)
+				(hide yes)
+			)
+		)
 		(pin "6"
 		)
@@
 			)
 		)
+		(property "FT Rotation Offset" "-90"
+			(at 229.87 78.74 0)
+			(effects
+				(font
+					(size 1.27 1.27)
+				)
+				(hide yes)
+			)
+		)
 		(pin "4"
 		)
@@
 			)
 		)
-		(property "Footprint" "Diode_SMD:D_SOD-123"
+		(property "Footprint" "Diode_SMD:D_SOD-323"
 			(at 162.56 111.76 90)
 			(effects

Commit message: Set LED resistors
Parts:
- R24, R33: value R -> 4.7k
- R25, R26: value 3.3k -> 1.2k
Changed lines of the file:
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@@
 			)
 		)
-		(property "Value" "3.3k"
+		(property "Value" "1.2k"
 			(at 66.04 147.3199 0)
 			(effects
@@
 		(fields_autoplaced yes)
 		(property "Reference" "R24"
-			(at 259.08 104.14 0)
+			(at 259.08 104.1399 0)
 			(effects
 				(font
@@
 			)
 		)
-		(property "Value" "R"
-			(at 259.08 106.68 0)
+		(property "Value" "4.7k"
+			(at 259.08 106.6799 0)
 			(effects
 				(font
@@
 		(fields_autoplaced yes)
 		(property "Reference" "R33"
-			(at 80.01 144.78 0)
+			(at 80.01 144.7799 0)
 			(effects
 				(font
@@
 			)
 		)
-		(property "Value" "R"
-			(at 80.01 147.32 0)
+		(property "Value" "4.7k"
+			(at 80.01 147.3199 0)
 			(effects
 				(font
@@
 			)
 		)
-		(property "Value" "3.3k"
+		(property "Value" "1.2k"
 			(at 274.32 106.6799 0)
 			(effects

Commit message: Switch to JST-PH connectors Add Sheet titles
Other:
- title: (none) -> Control MCU with Isolated USB-Serial Interface
Changed lines of the file:
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@@
 	(paper "A4")
 	(title_block
+		(title "Control MCU with Isolated USB-Serial Interface")
 		(rev "1.0")
+		(comment 1 "Through-hole connectors not to be installed as part of PCBA")
 	)
 	(text "~{TNOW} drives low when serial \ndata is being transmitted"

Commit message: Action review feedback
Parts:
- U6: value ADuM1201AR -> ADuM1201ARZ
Changed lines of the file:
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@@
 			)
 		)
-		(property "Value" "ADuM1201AR"
+		(property "Value" "ADuM1201ARZ"
 			(at 124.46 52.07 0)
 			(effects

Commit message: Omit tagconnect for BOM
Parts:
- J7: now left out of the parts list
Changed lines of the file:
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@@
 		(unit 1)
 		(exclude_from_sim no)
-		(in_bom yes)
+		(in_bom no)
 		(on_board yes)
 		(dnp no)
